Commit message: changed urdf and added moveit_config

File: src/ur_nova/urdf/ur_nova.urdf (robot description, URDF)
Before this commit: robot ur_nova, 20 links, 19 joints
Links:
- removed link base
- removed link base_link
- removed link ee_link
- removed link nova_carter
- removed link tool0
- removed link ur5_mount
- added link base_link_nova, mass 52.90850067138672; collision box size=0.67 0.35 0.26; visual mesh filename=package://nova_carter_description/meshes/chassis_link.stl
- link caster_swivel_left: geometry collision mesh filename=package://nova_carter_description/meshes/caster_swivel.stl; visual mesh filename=package://nova_carter_description/meshes/caster_swivel.stl
- link caster_swivel_right: geometry collision mesh filename=package://nova_carter_description/meshes/caster_swivel.stl; visual mesh filename=package://nova_carter_description/meshes/caster_swivel.stl
- link caster_wheel_left: geometry collision cylinder length=0.025 radius=0.0755; visual mesh filename=package://nova_carter_description/meshes/caster_wheel.stl
- link caster_wheel_right: geometry collision cylinder length=0.025 radius=0.0755; visual mesh filename=package://nova_carter_description/meshes/caster_wheel.stl
- link nova_carter_caster_frame_base: geometry collision mesh filename=package://nova_carter_description/meshes/caster_frame_base.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; visual mesh filename=package://nova_carter_description/meshes/caster_frame_base.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
Joints:
- removed joint base_link-base_fixed_joint
- removed joint ee_fixed_joint
- removed joint nova_mount_joint
- removed joint nova_ur_joint
- removed joint wrist_3_link-tool0_fixed_joint
- joint joint_caster_base: parent nova_carter -> base_link_nova
- joint joint_wheel_left: parent nova_carter -> base_link_nova
- joint joint_wheel_right: parent nova_carter -> base_link_nova
- joint nova_carter_joint: child nova_carter -> base_link_nova
- joint shoulder_pan_joint: origin xyz=0.0 0.0 0.089159 rpy=0.0 0.0 0.0 -> xyz=-0.23 0 0.55 rpy=0 0 0; parent base_link -> base_link_nova
